Commit message: add toy example with 2link robot, update files to handle more than just iiwa

File: robot_data/2link_robot.urdf (robot description, URDF)
Before this commit: robot 2link_robot, 4 links, 3 joints
Links:
- link endEffector: mass None -> 0
Joints:
- joint baseHinge: limit (none) -> lower=-2.9670597283903604 upper=2.9670597283903604 effort=20 velocity=10; origin (none) -> xyz=0 0 0.15 rpy=0 0 0
- joint interArm: limit (none) -> lower=-2.9670597283903604 upper=2.9670597283903604 effort=300 velocity=10

Commit message: Work in progress tests

File: robot_data/2link_robot.urdf (robot description, URDF)
Before this commit: robot 2link_robot, 4 links, 3 joints
Joints:
- joint baseHinge: type continuous -> revolute
- joint interArm: limit lower=-2.9670597283903604 upper=2.9670597283903604 effort=300 velocity=10 -> lower=-2.9670597283903604 upper=2.9670597283903604 effort=20 velocity=10; type continuous -> revolute

Commit message: 2 link arm passes tests

File: robot_data/2link_robot.urdf (robot description, URDF)
Before this commit: robot 2link_robot, 4 links, 3 joints
Joints:
- joint ee_joint: origin xyz=1 0 0 rpy=0 0 0 -> xyz=0 0 0.05 rpy=0 0 0
