Commit message: debugging

File: robot_data/panda_description/urdf/panda.urdf (robot description, URDF)
Before this commit: robot panda, 12 links, 11 joints
Links:
- link panda_link8: mass None -> 0

Commit message: updating panda description

File: robot_data/panda_description/urdf/panda.urdf (robot description, URDF)
Before this commit: robot panda, 12 links, 11 joints
Links:
- added link panda_virtual_ee_link, mass 0.0
- link panda_hand: mass None -> .81
- link panda_leftfinger: mass None -> 0.1
- link panda_link0: mass None -> 2.9
- link panda_link1: mass None -> 2.7
- link panda_link2: mass None -> 2.73
- link panda_link3: mass None -> 2.04
- link panda_link4: mass None -> 2.08
- link panda_link5: mass None -> 3
- link panda_link6: mass None -> 1.3
- link panda_link7: mass None -> .2
- link panda_link8: mass 0 -> 0.0
- link panda_rightfinger: mass None -> 0.1
Joints:
- added joint panda_virtual_ee_joint: type fixed, parent panda_hand, child panda_virtual_ee_link, origin xyz=0 0 0.105 rpy=0 0 0
