Commit message: adding fetch arm without gripper

File: diff_robot_data/fetch_description/urdf/fetch_arm_no_gripper.urdf (robot description, URDF)
Before this commit: robot fetch, 12 links, 11 joints
Links:
- removed link gripper_link
- removed link l_gripper_finger_link
- removed link r_gripper_finger_link
Joints:
- removed joint gripper_axis
- removed joint l_gripper_finger_joint
- removed joint r_gripper_finger_joint
- joint virtual_ee_joint: parent gripper_link -> wrist_roll_link
