Commit message: Add jaco urdfs

File: diff_robot_data/kinova_description/urdf/jaco.urdf (robot description, URDF)
Before this commit: robot j2n6s300, 16 links, 15 joints
Links:
- removed link world
Joints:
- removed joint connect_root_and_world

File: diff_robot_data/kinova_description/urdf/jaco_clean.urdf (robot description, URDF)
Before this commit: robot j2n6s300, 16 links, 15 joints
Links:
- removed link world
- added link j2n6s300_link_ee, mass 0
Joints:
- removed joint connect_root_and_world
- added joint j2n6s300_joint_ee: type fixed, parent j2n6s300_end_effector, child j2n6s300_link_ee, origin xyz=0 0 0.045 rpy=0 0 0
